File: magical555vco.kicad_pcb (KiCad board)
At the start: 2 copper layers, 40.3 x 128.5 mm, 14 parts, among them J1 Eurorack_Power_16pin_Unshroud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, J2 OUTPUT 1, J3 INPUT 1, U1 NE555P, U2 TL074

Commit message: 2 modules, potmeter
Parts:
- added C3: 100nF, Capacitor_THT:C_Disc_D5.0mm_W2.5mm_P5.00mm, F.Cu at (120.8, 111.3)
- added C4: 10nF, Capacitor_THT:C_Disc_D5.0mm_W2.5mm_P5.00mm, F.Cu at (148.7, 111.3)
- added D3: 1N4148, Diode_THT:D_DO-35_SOD27_P7.62mm_Horizontal, F.Cu at (123.3, 127.9)
- added D4: 1N4148, Diode_THT:D_DO-35_SOD27_P7.62mm_Horizontal, F.Cu at (151.3, 127.9)
- added J4: INPUT 1, Connector_Audio:Jack_3.5mm_QingPu_WQP-PJ398SM_Vertical_CircularHoles, F.Cu at (123.3, 93.6)
- added J5: OUTPUT 1, Connector_Audio:Jack_3.5mm_QingPu_WQP-PJ398SM_Vertical_CircularHoles, F.Cu at (151.3, 93.6)
- added R6: 10k, Resistor_THT:R_Axial_DIN0204_L3.6mm_D1.6mm_P7.62mm_Horizontal, F.Cu at (135.3, 102.5)
- added R7: 10k, Resistor_THT:R_Axial_DIN0204_L3.6mm_D1.6mm_P7.62mm_Horizontal, F.Cu at (139.3, 102.5)
- added R8: 10k, Resistor_THT:R_Axial_DIN0204_L3.6mm_D1.6mm_P7.62mm_Horizontal, F.Cu at (143.3, 102.5)
- added RV1: B1M, Potentiometer_THT:Potentiometer_Alps_RK09K_Single_Vertical, F.Cu at (134.7, 89.6)
- added RV2: B1M, Potentiometer_THT:Potentiometer_Alps_RK09K_Single_Vertical, F.Cu at (135.3, 128.9)
- added U4: NE555P, Package_DIP:DIP-8_W7.62mm, F.Cu at (133.4, 113.3)
- R2: value 100k -> 10k
- moved R2 44.6 mm to (131.3, 102.5)
- moved R1 2.82 mm to (143.3, 62.3)
- moved U1 2.41 mm to (133.7, 73.4)
- moved C2 2.41 mm to (147.3, 71.0)
- moved D1 2.41 mm to (120.5, 77.1)
- moved J2 2.41 mm to (151.3, 54.8)
- moved J3 2.41 mm to (123.3, 54.9)
- moved C1 2.41 mm to (122.3, 71.2)
- moved D2 2.41 mm to (145.7, 77.1)
- moved R5 2.33 mm to (139.3, 62.3)
- moved R3 2.26 mm to (131.3, 62.3)
- moved R4 2.13 mm to (135.3, 62.3)
Connections:
- R2 pad 1: Net-(U1-THR) -> Net-(U2C-+)
- R2 pad 2: Net-(U1-Q) -> Net-(J4-PadT)
- U2 pad 10: (no net) -> Net-(U2C-+)
- U2 pad 12: (no net) -> GND
- U2 pad 13: (no net) -> Net-(U2D--)
- U2 pad 14: (no net) -> Net-(J5-PadT)
- U2 pad 8: (no net) -> Net-(D3-A)
- U2 pad 9: (no net) -> Net-(D3-A)
Routing:
- net GND: track 0.00 -> 237.9 mm
- net +5V: track 0.00 -> 138.4 mm
- net Net-(D1-A): track 0.00 -> 117.4 mm
- net +12V: track 0.00 -> 113.7 mm
- net Net-(J2-PadT): track 0.00 -> 108.3 mm
- net -12V: track 0.00 -> 104.8 mm
- net Net-(U2B-+): track 0.00 -> 98.1 mm
- net Net-(U2A--): track 0.00 -> 97.6 mm
- net Net-(D3-A): track 0.00 -> 72.1 mm
- net Net-(U2D--): track 0.00 -> 66.2 mm
- net Net-(J5-PadT): track 0.00 -> 56.4 mm
- net Net-(U2C-+): track 0.00 -> 50.0 mm
- net Net-(U4-THR): track 0.00 -> 41.2 mm
- net Net-(U1-Q): track 0.00 -> 36.7 mm
- net Net-(U4-Q): track 0.00 -> 36.1 mm
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- added copper zone on B.Cu, net GND
- added copper zone on F.Cu, net GND
Other:
- board text added: "v0.1"

Commit message: v0.2
Parts:
- added R10: 10k, Resistor_THT:R_Axial_DIN0204_L3.6mm_D1.6mm_P7.62mm_Horizontal, F.Cu at (124.5, 133.3)
- added R11: 10k, Resistor_THT:R_Axial_DIN0204_L3.6mm_D1.6mm_P7.62mm_Horizontal, F.Cu at (143.5, 133.3)
- added R12: 10k, Resistor_THT:R_Axial_DIN0204_L3.6mm_D1.6mm_P7.62mm_Horizontal, F.Cu at (124.5, 81.3)
- added R9: 10k, Resistor_THT:R_Axial_DIN0204_L3.6mm_D1.6mm_P7.62mm_Horizontal, F.Cu at (149.9, 88.9)
- R1, R3, R7, R8: value 10k -> 20k
Connections:
- R1 pad 1: Net-(U2B-+) -> Net-(U2A--)
- R2 pad 1: Net-(U2C-+) -> Net-(D1-A)
- R2 pad 2: Net-(J4-PadT) -> Net-(U2A--)
- R3 pad 1: Net-(J2-PadT) -> Net-(U2A-+)
- R3 pad 2: Net-(U2A--) -> +5V
- R4 pad 1: Net-(U2A--) -> Net-(U2A-+)
- R4 pad 2: Net-(U1-Q) -> GND
- R5 pad 1: +5V -> Net-(J2-PadT)
- R5 pad 2: Net-(U2B-+) -> Net-(U2B--)
- R6 pad 1: +5V -> Net-(U2B--)
- R6 pad 2: Net-(U2C-+) -> +5V
- R7 pad 1: Net-(U2D--) -> Net-(U2C--)
- R7 pad 2: Net-(U4-Q) -> Net-(J4-PadT)
- R8 pad 1: Net-(J5-PadT) -> Net-(U2C-+)
- R8 pad 2: Net-(U2D--) -> +5V
- RV2 pad 3: Net-(U4-Q) -> Net-(U2D-+)
- U2 pad 1: Net-(J2-PadT) -> Net-(D1-A)
- U2 pad 12: GND -> Net-(U2D-+)
- U2 pad 3: GND -> Net-(U2A-+)
- U2 pad 5: Net-(U2B-+) -> Net-(U1-Q)
- U2 pad 6: Net-(D1-A) -> Net-(U2B--)
- U2 pad 7: Net-(D1-A) -> Net-(J2-PadT)
- U2 pad 9: Net-(D3-A) -> Net-(U2C--)
- U4 pad 3: Net-(U4-Q) -> Net-(U2D-+)
Routing:
- net Net-(U2B--): track 0.00 -> 105.4 mm
- net Net-(U2B-+): track 98.1 -> 0.00 mm
- net Net-(U2A-+): track 0.00 -> 91.7 mm
- net Net-(U2C--): track 0.00 -> 64.8 mm
- net Net-(U1-Q): track 36.7 -> 80.0 mm
- net Net-(J5-PadT): track 56.4 -> 98.4 mm
- net Net-(U4-Q): track 36.1 -> 0.00 mm
- net GND: track 237.9 -> 208.0 mm
- net Net-(U2D-+): track 0.00 -> 29.5 mm
- net +5V: track 138.4 -> 155.2 mm
- net Net-(D3-A): track 72.1 -> 84.3 mm
- net Net-(U2D--): track 66.2 -> 78.4 mm
- net Net-(J2-PadT): track 108.3 -> 97.4 mm
- net Net-(U2C-+): track 50.0 -> 60.9 mm
- net Net-(U2A--): track 97.6 -> 108.1 mm
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Other:
- board text added: "v0.2"
- board text removed: "v0.1"
