File: magical555vco.kicad_sch (KiCad schematic)
At the start: 14 parts, among them J1 Eurorack_Power_16pin_Unshroud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, J2 OUTPUT 1, J3 INPUT 1, U1 NE555P, U2 TL074

Commit message: 2 modules, potmeter
Parts:
- added C3: 100nF, Capacitor_THT:C_Disc_D5.0mm_W2.5mm_P5.00mm, symbol Device:C
- added C4: 10nF, Capacitor_THT:C_Disc_D5.0mm_W2.5mm_P5.00mm, symbol Device:C
- added D3, D4: 1N4148, Diode_THT:D_DO-35_SOD27_P7.62mm_Horizontal, symbol Diode:1N4148
- added J4: INPUT 1, Connector_Audio:Jack_3.5mm_QingPu_WQP-PJ398SM_Vertical_CircularHoles, symbol Connector:AudioJack2
- added J5: OUTPUT 1, Connector_Audio:Jack_3.5mm_QingPu_WQP-PJ398SM_Vertical_CircularHoles, symbol Connector:AudioJack2
- added R6, R7, R8: 10k, Resistor_THT:R_Axial_DIN0204_L3.6mm_D1.6mm_P7.62mm_Horizontal, symbol Device:R
- added RV1, RV2: B1M, Potentiometer_THT:Potentiometer_Alps_RK09K_Single_Vertical, symbol Device:R_Potentiometer
- added unit 3 of U2
- added unit 4 of U2
- added U4: NE555P, Package_DIP:DIP-8_W7.62mm, symbol Timer:NE555P
- R2: value 100k -> 10k
Connections:
- net +5V: now also D3.1 (K), R6.1, U4.4 (R), U4.8 (VCC)
- net GND: now also C3.1, C4.1, D4.2 (A), J4.S, J5.S, U2.12 (+), U4.1 (GND)
- net at C1.2, U1.2 (TR), U1.6 (THR): now also RV1.2; no longer R2.1
- net at R4.2, U1.3 (Q): now also RV1.3; no longer R2.2
- new net: C4.2, RV2.2, U4.2 (TR), U4.6 (THR)
- new net: R7.2, RV2.3, U4.3 (Q)
- new net: C3.2, D3.2 (A), D4.1 (K), U2.8, U2.9 (-), U4.5 (CV)
- new net: J5.T, R8.1, U2.14
- new net: R7.1, R8.2, U2.13 (-)
- new net: R2.1, R6.2, U2.10 (+)
- new net: J4.T, R2.2

Commit message: v0.2
Parts:
- added R10, R11, R12, R9: 10k, Resistor_THT:R_Axial_DIN0204_L3.6mm_D1.6mm_P7.62mm_Horizontal, symbol Device:R
- R1, R3, R7, R8: value 10k -> 20k
Connections:
- net +5V: now also R3.2, R6.2, R8.2, R11.2; no longer R5.1, R6.1
- net GND: now also R4.2, R9.2; no longer U2.12 (+), U2.3 (+)
- net at C2.2, D1.2 (A), D2.1 (K)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: now also R2.1, U2.1; no longer U2.6 (-), U2.7
- net at RV2.3, U4.3 (Q): now also U2.12 (+); no longer R7.2
- net at C3.2, D3.2 (A), D4.1 (K)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: now also R10.1; no longer U2.9 (-)
- net at RV1.3, U1.3 (Q): now also U2.5 (+); no longer R4.2
- net at J5.T, U2.14: now also R12.1; no longer R8.1
- net at R2.2: now also R1.1, U2.2 (-); no longer J4.T
- new net: J2.T, R5.1, U2.7
- new net: R5.2, R6.1, U2.6 (-)
- new net: R11.1, R12.2, U2.13 (-)
- new net: R10.2, R7.1, U2.9 (-)
- new net: J4.T, R7.2
- new net: R8.1, R9.1, U2.10 (+)
- new net: R3.1, R4.1, U2.3 (+)
Other:
- note added: "transform 0...5V into -5...+5V"
- note removed: "invert signal"
- moved on the sheet: J2

Commit message: meta
Other:
- company: (none) -> www.vanheusden.com
- title: (none) -> Magical555VCO
Changed lines of the file:
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@@
 (kicad_sch (version 20230121) (generator eeschema)
   (paper "A4")
+  (title_block
+    (title "Magical555VCO")
+    (date "2023-10-28")
+    (rev "0.2")
+    (company "www.vanheusden.com")
+  )
   (junction (at 191.77 44.45) (diameter 0) (color 0 0 0 0)
   )
